File: weirdo.kicad_pcb (KiCad board)
At the start: 2 copper layers, 194 x 103.8 mm, 89 parts, among them J1 Conn_01x08, J2 Conn_01x08, U2 ProMicro

Commit message: hoah.
Parts:
- added switch33: switch, footprints:1u-single, F.Cu at (136.3, 96.4)
- added switch34: switch, footprints:1u-single, F.Cu at (98.7, 96.3)
Routing:
- net Net-(diode32-Pad2): track 16.6 -> 28.9 mm
- net COLB4: track 164.3 -> 175.0 mm
- net COLA3: track 169.5 -> 180.1 mm
- net Net-(diode4-Pad2): track 14.2 -> 17.2 mm
